Commit message: type:fix    fix a bug that gazebo model is not properly launched

File: urdf/robot.xacro (robot description, xacro)
@@ -9,3 +9,5 @@
   <xacro:include filename="$(find xbot2_description)/urdf/sick_tim.urdf.xacro" />
   <xacro:sick_tim571 name="laser" ros_topic="scan"   />
+  <xacro:include filename="$(find xbot2_description)/urdf/xbot2.gazebo.xacro" />
+  <xacro:include filename="$(find xbot2_description)/urdf/sick_tim.gazebo.xacro" />
 </robot>

File: urdf/sick_tim.gazebo.xacro (robot description, xacro)
@@ -1,14 +1,3 @@
-<robot xmlns:xacro="http://www.ros.org/wiki/xacro" name="xbot2" >
-  <!-- Base is modeled as a big tub sitting on floor, with two wheels -->
-  <gazebo reference="base_link">
-    <kp>100000000.0</kp>
-    <kd>10.0</kd>
-    <mu1>0.1</mu1>
-    <mu2>0.1</mu2>
-    <fdir1>1 0 0</fdir1>
-    <maxVel>10.0</maxVel>
-    <minDepth>0.0005</minDepth>
-    <material>Gazebo/Black</material>
-  </gazebo>
+<robot xmlns:xacro="http://www.ros.org/wiki/xacro" name="sick_tim" >
   <!-- SICK TIM571 (25m Range) -->
   <gazebo reference="laser">

Commit message: type: fix 1.started to use new xbot2 model(.dae) 2.modified laser model 3.modified gazebo laser plugin

File: urdf/robot.xacro (robot description, xacro)
@@ -9,5 +9,5 @@
   <xacro:include filename="$(find xbot2_description)/urdf/sick_tim.urdf.xacro" />
   <xacro:sick_tim571 name="laser" ros_topic="scan"   />
-  <xacro:include filename="$(find xbot2_description)/urdf/xbot2.gazebo.xacro" />
-  <xacro:include filename="$(find xbot2_description)/urdf/sick_tim.gazebo.xacro" />
+  <!--xacro:include filename="$(find xbot2_description)/urdf/xbot2.gazebo.xacro" /-->
+  <!--xacro:include filename="$(find xbot2_description)/urdf/sick_tim.gazebo.xacro" /-->
 </robot>

File: urdf/sick_tim.gazebo.xacro (robot description, xacro)
@@ -28,5 +28,5 @@
       </ray>
       <plugin name="gazebo_ros_base_sick_controller" filename="libgazebo_ros_laser.so">
-        <topicName>/base_scan</topicName>
+        <topicName>/scan</topicName>
         <frameName>laser_link</frameName>
       </plugin>

File: urdf/sick_tim.urdf.xacro (robot description, xacro)
@@ -18,5 +18,5 @@
   <xacro:macro name="sick_tim571" params="name ros_topic">
     <xacro:sick_tim name="${name}" ros_topic="${ros_topic}"
-      length="0.06" width="0.06" height="0.086" mass="0.250" z_offset="0.05"
+      length="0.06" width="0.06" height="0.086" mass="0.250" z_offset="0.02"
       min_range="0.05" max_range="25.0"
       mesh="package://xbot2_description/meshes/sick_tim571.stl" />
@@ -55,5 +55,5 @@
   <xacro:macro name="sick_tim_laser_gazebo_v0" params="name link ros_topic update_rate min_angle max_angle min_range max_range">
     <gazebo reference="${link}">
-      <material value="Gazebo/Blue" />
+      <material value="Gazebo/LightWood" />
       <sensor type="ray" name="${name}">
         <always_on>true</always_on>
@@ -64,5 +64,5 @@
           <scan>
             <horizontal>
-              <samples>271</samples>
+              <samples>810</samples>
               <resolution>1</resolution>
               <min_angle>${min_angle}</min_angle>

File: urdf/xbot2.gazebo.xacro (robot description, xacro)
@@ -9,5 +9,5 @@
     <maxVel>10.0</maxVel>
     <minDepth>0.0005</minDepth>
-    <material>Gazebo/Black</material>
+    <material>PR2/Grey0</material>
   </gazebo>
   <!-- SICK TIM571 (25m Range) -->

File: urdf/xbot2.urdf.xacro (robot description, xacro)
@@ -23,7 +23,4 @@
         <mesh filename="package://xbot2_description/meshes/base_link.dae" />
       </geometry>
-      <material name="">
-        <texture filename="package://xbot2_description/meshes/black_felt.png" />
-      </material>
     </visual>
     <collision>
@@ -39,5 +36,5 @@
     <parent link="base_link"/>
     <child link="laser_mount_link"/>
-    <origin rpy="0 3.1416 3.1416" xyz=".08 -0.03 .253"/>
+    <origin rpy="0 3.1416 3.1416" xyz=".118 0 .253"/>
   </joint>
   </xacro:macro>

Commit message: type: fix add two fake continuous wheels to simulate going forward. the next step is to seperate xbot2 wheels and body.

File: urdf/robot.xacro (robot description, xacro)
@@ -5,9 +5,9 @@
   xmlns:xacro="http://ros.org/wiki/xacro"
   name="sick_tim">
+  <xacro:include filename="$(find xbot2_description)/urdf/xbot2.gazebo" />
   <xacro:include filename="$(find xbot2_description)/urdf/xbot2.urdf.xacro" />
   <xacro:xbot2_base/>
   <xacro:include filename="$(find xbot2_description)/urdf/sick_tim.urdf.xacro" />
   <xacro:sick_tim571 name="laser" ros_topic="scan"   />
-  <!--xacro:include filename="$(find xbot2_description)/urdf/xbot2.gazebo.xacro" /-->
   <!--xacro:include filename="$(find xbot2_description)/urdf/sick_tim.gazebo.xacro" /-->
 </robot>

File: urdf/xbot2.urdf.xacro (robot description, xacro)
@@ -38,4 +38,66 @@
     <origin rpy="0 3.1416 3.1416" xyz=".118 0 .253"/>
   </joint>
+  <link name="left_wheel">
+    <collision name="collision">
+      <origin xyz="0 0 0" rpy="0 1.5707 1.5707"/>
+      <geometry>
+        <cylinder radius="0.1" length="0.02"/>
+      </geometry>
+    </collision>
+    <visual name="left_wheel_visual">
+      <origin xyz="0 0 0" rpy="0 1.5707 1.5707"/>
+      <geometry>
+        <cylinder radius="0.1" length="0.02"/>
+      </geometry>
+    </visual>
+    <inertial>
+      <origin xyz="0 0 0" rpy="0 1.5707 1.5707"/>
+      <mass value="5"/>
+      <cylinder_inertia m="5" r="0.1" h="0.05"/>
+      <inertia
+        ixx="1.0" ixy="0.0" ixz="0.0"
+        iyy="1.0" iyz="0.0"
+        izz="1.0"/>
+    </inertial>
+  </link>
+  <link name="right_wheel">
+    <collision name="collision">
+      <origin xyz="0 0 0" rpy="0 1.5707 1.5707"/>
+      <geometry>
+        <cylinder radius="0.1" length="0.02"/>
+      </geometry>
+    </collision>
+    <visual name="right_wheel_visual">
+      <origin xyz="0 0 0" rpy="0 1.5707 1.5707"/>
+      <geometry>
+        <cylinder radius="0.1" length="0.02"/>
+      </geometry>
+    </visual>
+    <inertial>
+      <origin xyz="0 0 0" rpy="0 1.5707 1.5707"/>
+      <mass value="5"/>
+      <cylinder_inertia m="5" r="0.1" h="0.05"/>
+      <inertia
+        ixx="1.0" ixy="0.0" ixz="0.0"
+        iyy="1.0" iyz="0.0"
+        izz="1.0"/>
+    </inertial>
+  </link>
+  <joint type="continuous" name="left_wheel_hinge">
+    <origin xyz="0 0.3 0.08" rpy="0 0 0"/>
+    <child link="left_wheel"/>
+    <parent link="base_link"/>
+    <axis xyz="0 1 0" rpy="0 0 0"/>
+    <limit effort="100" velocity="100"/>
+    <joint_properties damping="0.0" friction="0.0"/>
+  </joint>
+  <joint type="continuous" name="right_wheel_hinge">
+    <origin xyz="0 -0.3 0.08" rpy="0 0 0"/>
+    <child link="right_wheel"/>
+    <parent link="base_link"/>
+    <axis xyz="0 1 0" rpy="0 0 0"/>
+    <limit effort="100" velocity="100"/>
+    <joint_properties damping="0.0" friction="0.0"/>
+  </joint>
   </xacro:macro>
 </robot>

Commit message: type: feat add RGBD camera model and simulation lib to gazebo

File: urdf/robot.xacro (robot description, xacro)
@@ -5,9 +5,10 @@
   xmlns:xacro="http://ros.org/wiki/xacro"
   name="sick_tim">
-  <xacro:include filename="$(find xbot2_description)/urdf/xbot2.gazebo" />
-  <xacro:include filename="$(find xbot2_description)/urdf/xbot2.urdf.xacro" />
-  <xacro:xbot2_base/>
   <xacro:include filename="$(find xbot2_description)/urdf/sick_tim.urdf.xacro" />
   <xacro:sick_tim571 name="laser" ros_topic="scan"   />
+  <xacro:include filename="$(find xbot2_description)/urdf/materials.xacro" />
+  <xacro:include filename="$(find xbot2_description)/urdf/xbot2.urdf.xacro" />
+  <xacro:include filename="$(find xbot2_description)/urdf/xbot2.gazebo" />
+  <xacro:xbot2_base/>
   <!--xacro:include filename="$(find xbot2_description)/urdf/sick_tim.gazebo.xacro" /-->
 </robot>

File: urdf/sick_tim.urdf.xacro (robot description, xacro)
@@ -34,6 +34,6 @@
           <mesh filename="${mesh}" />
         </geometry>
-        <material name="blue" >
-          <color rgba="0 0 1 1" />
+        <material name="lightblue">
+          <color rgba=".5 .5 .7 .8" />
         </material>
       </visual>

File: urdf/xbot2.urdf.xacro (robot description, xacro)
@@ -101,11 +101,12 @@
       <origin xyz="0 0 0" rpy="0 0 1.5708" />
       <geometry>
-        <mesh filename="package://xbot2_description/meshes/yaw_platform.dae" />
+        <mesh filename="package://xbot2_description/meshes/yaw_platform.stl" />
       </geometry>
+      <material name="grey"/>
     </visual>
     <collision>
       <origin xyz="0 0 0" rpy="0 0 1.5708" />
       <geometry>
-        <mesh filename="package://xbot2_description/meshes/yaw_platform.dae" />
+        <mesh filename="package://xbot2_description/meshes/yaw_platform.stl" />
       </geometry>
     </collision>
@@ -117,4 +118,5 @@
     <origin rpy="0 0 0" xyz="0 0 1.07"/>
     <limit effort="100" velocity="100" lower="-1.57" upper="1.57" />
+    <dynamics damping="0.0" friction="5.0"/>
   </joint>
   <link name="pitch_platform">
@@ -129,4 +131,5 @@
         <mesh filename="package://xbot2_description/meshes/pitch_platform.stl" />
       </geometry>
+      <material name="grey"/>
     </visual>
     <collision>
@@ -143,4 +146,5 @@
     <origin rpy="0 0 0" xyz="0 0 .02"/>
     <limit effort="100" velocity="100" lower="-1.57" upper="1.57" />
+    <dynamics damping="0.0" friction="5.0"/>
   </joint>
   <!-- Camera -->
@@ -157,5 +161,5 @@
         <mesh filename="package://xbot2_description/meshes/xtion_pro_camera.dae" />
       </geometry>
-      <material name="red"/>
+      <material name="gray"/>
     </visual>
     <inertial>
@@ -167,5 +171,5 @@
   <joint name="camera_joint" type="fixed">
     <axis xyz="0 1 0" />
-    <origin xyz="0 0 0" rpy="0 0 0"/>
+    <origin xyz="0 0 .08" rpy="0 0 0"/>
     <parent link="pitch_platform"/>
     <child link="camera_link"/>
