Commit message: replace xbot_base with dae model

File: urdf/sick_tim.urdf.xacro (robot description, xacro)
@@ -18,6 +18,6 @@
   <xacro:macro name="sick_tim571" params="name ros_topic">
     <xacro:sick_tim name="${name}" ros_topic="${ros_topic}"
-      length="0.06" width="0.06" height="0.086" mass="0.250" z_offset="0.06296"
-      min_range="0.05" max_range="10.0"
+      length="0.06" width="0.06" height="0.086" mass="0.250" z_offset="0.05"
+      min_range="0.05" max_range="25.0"
       mesh="package://xbot2_description/meshes/sick_tim571.stl" />
   </xacro:macro>
@@ -77,5 +77,5 @@
         </ray>
         <plugin name="gazebo_ros_${name}_controller" filename="libgazebo_ros_laser.so">
-          <gaussianNoise>0.005</gaussianNoise>
+          <gaussianNoise>0.01</gaussianNoise>
           <alwaysOn>true</alwaysOn>
           <updateRate>${update_rate}</updateRate>

File: urdf/xbot2.gazebo.xacro (robot description, xacro)
@@ -32,5 +32,5 @@
         </range>
         <noise>
-          <!-- Noise parameters based on spec for SICK TIM561 (10m version) -->
+          <!-- Noise parameters based on spec for SICK TIM571 (25m version) -->
           <type>gaussian</type>
           <mean>0.0</mean>
@@ -38,5 +38,5 @@
         </noise>
       </ray>
-      <plugin name="gazebo_ros_base_hokuyo_controller" filename="libgazebo_ros_laser.so">
+      <plugin name="gazebo_ros_base_sick_controller" filename="libgazebo_ros_laser.so">
         <topicName>/base_scan</topicName>
         <frameName>laser_link</frameName>
@@ -48,7 +48,3 @@
     <material>Gazebo/Red</material>
   </gazebo>
-  <!-- Load the plugin -->
-  <gazebo>
-    <plugin name="fetch_gazebo_plugin" filename="libfetch_gazebo_plugin.so"/>
-  </gazebo>
 </robot>

File: urdf/xbot2.urdf.xacro (robot description, xacro)
@@ -21,5 +21,5 @@
       <origin xyz="0 0 0" rpy="0 0 0" />
       <geometry>
-        <mesh filename="package://xbot2_description/meshes/base_link.STL" />
+        <mesh filename="package://xbot2_description/meshes/base_link.dae" />
       </geometry>
       <material name="">
@@ -30,5 +30,5 @@
       <origin xyz="0 0 0" rpy="0 0 0" />
       <geometry>
-        <mesh filename="package://xbot2_description/meshes/base_link.STL" />
+        <mesh filename="package://xbot2_description/meshes/base_link.dae" />
       </geometry>
     </collision>
@@ -39,5 +39,5 @@
     <parent link="base_link"/>
     <child link="laser_mount_link"/>
-    <origin rpy="0 0 0" xyz="0 0 .2"/>
+    <origin rpy="0 3.1416 3.1416" xyz=".08 -0.03 .253"/>
   </joint>
   </xacro:macro>

Commit message: type: feat add yaw and pitch platforms on top of xbot base link

File: urdf/sick_tim.urdf.xacro (robot description, xacro)
@@ -51,5 +51,7 @@
       </inertial>
     </link>
-    <xacro:sick_tim_laser_gazebo_v0 name="${name}" link="${name}" ros_topic="${ros_topic}" update_rate="15.0" min_angle="-2.357" max_angle="2.357" min_range="${min_range}" max_range="${max_range}"/>
+    <xacro:sick_tim_laser_gazebo_v0 name="${name}" link="${name}" ros_topic="${ros_topic}"
+    update_rate="15.0" min_angle="-2.357" max_angle="2.357" min_range="${min_range}" max_range="${max_range}"/>
+    <!--update_rate=15.0-->
   </xacro:macro>
   <xacro:macro name="sick_tim_laser_gazebo_v0" params="name link ros_topic update_rate min_angle max_angle min_range max_range">
@@ -60,9 +62,9 @@
         <update_rate>${update_rate}</update_rate>
         <pose>0 0 0 0 0 0</pose>
-        <visualize>false</visualize>
+        <visualize>true</visualize>
         <ray>
           <scan>
             <horizontal>
-              <samples>810</samples>
+              <samples>810</samples>  <!-- 810 -->
               <resolution>1</resolution>
               <min_angle>${min_angle}</min_angle>

File: urdf/xbot2.urdf.xacro (robot description, xacro)
@@ -61,4 +61,11 @@
     </inertial>
   </link>
+  <joint type="continuous" name="left_wheel_hinge">
+    <axis xyz="0 1 0" rpy="0 0 0"/>
+    <origin xyz="0 0.3 0.08" rpy="0 0 0"/>
+    <parent link="base_link"/>
+    <child link="left_wheel"/>
+    <joint_properties damping="0.0" friction="0.0"/>
+  </joint>
   <link name="right_wheel">
     <collision name="collision">
@@ -84,19 +91,62 @@
     </inertial>
   </link>
-  <joint type="continuous" name="left_wheel_hinge">
-    <origin xyz="0 0.3 0.08" rpy="0 0 0"/>
-    <child link="left_wheel"/>
+  <joint type="continuous" name="right_wheel_hinge">
+    <axis xyz="0 1 0" rpy="0 0 0"/>
+    <origin xyz="0 -0.3 0.08" rpy="0 0 0"/>
     <parent link="base_link"/>
-    <axis xyz="0 1 0" rpy="0 0 0"/>
-    <limit effort="100" velocity="100"/>
+    <child link="right_wheel"/>
     <joint_properties damping="0.0" friction="0.0"/>
   </joint>
-  <joint type="continuous" name="right_wheel_hinge">
-    <origin xyz="0 -0.3 0.08" rpy="0 0 0"/>
-    <child link="right_wheel"/>
+  <link name="yaw_platform">
+    <inertial>
+      <origin  xyz="-0.0033678 -0.047443 0.62953" rpy="0 0 0" />
+      <mass value=".109" />
+      <inertia ixx="0.82582" ixy="-0.0019603" ixz="-0.00043035" iyy="0.92115" iyz="0.0013243" izz="0.2601" />
+    </inertial>
+    <visual>
+      <origin xyz="0 0 0" rpy="0 0 1.5708" />
+      <geometry>
+        <mesh filename="package://xbot2_description/meshes/yaw_platform.dae" />
+      </geometry>
+    </visual>
+    <collision>
+      <origin xyz="0 0 0" rpy="0 0 1.5708" />
+      <geometry>
+        <mesh filename="package://xbot2_description/meshes/yaw_platform.dae" />
+      </geometry>
+    </collision>
+  </link>
+  <joint name="base_to_yaw_platform" type="revolute">
+    <axis xyz="0 0 1"/>
     <parent link="base_link"/>
-    <axis xyz="0 1 0" rpy="0 0 0"/>
-    <limit effort="100" velocity="100"/>
-    <joint_properties damping="0.0" friction="0.0"/>
+    <child link="yaw_platform"/>
+    <origin rpy="0 0 0" xyz="0 0 1.07"/>
+    <limit effort="100" velocity="100" lower="-1.57" upper="1.57" />
+  </joint>
+  <link name="pitch_platform">
+    <inertial>
+      <origin  xyz="-0.0033678 -0.047443 0.62953" rpy="0 0 0" />
+      <mass value=".109" />
+      <inertia ixx="0.82582" ixy="-0.0019603" ixz="-0.00043035" iyy="0.92115" iyz="0.0013243" izz="0.2601" />
+    </inertial>
+    <visual>
+      <origin xyz="0 0 0" rpy="0 3.1416 1.5708" />
+      <geometry>
+        <mesh filename="package://xbot2_description/meshes/pitch_platform.dae" />
+      </geometry>
+    </visual>
+    <collision>
+      <origin xyz="0 0 0" rpy="0 3.1416 1.5708" />
+      <geometry>
+        <mesh filename="package://xbot2_description/meshes/pitch_platform.dae" />
+      </geometry>
+    </collision>
+  </link>
+  <joint name="yaw_to_pitch_platform" type="revolute">
+    <axis xyz="0 1 0"/>
+    <parent link="yaw_platform"/>
+    <child link="pitch_platform"/>
+    <origin rpy="0 0 0" xyz="0 0 .08"/>
+    <limit effort="100" velocity="100" lower="-1.57" upper="1.57" />
   </joint>
   </xacro:macro>

Commit message: type: feat 1. add dynamics(friction, resilience, damp) to the robot 2. seperate the base into two parts: wheels and the main body 3. add xbot2_control.yaml configuration which receives message to control the joint and speed

File: urdf/sick_tim.urdf.xacro (robot description, xacro)
@@ -62,5 +62,5 @@
         <update_rate>${update_rate}</update_rate>
         <pose>0 0 0 0 0 0</pose>
-        <visualize>true</visualize>
+        <visualize>false</visualize>
         <ray>
           <scan>

File: urdf/xbot2.urdf.xacro (robot description, xacro)
@@ -14,7 +14,7 @@
   <link name="base_link">
     <inertial>
-      <origin  xyz="-0.0033678 -0.047443 0.62953" rpy="0 0 0" />
-      <mass value="12.609" />
-      <inertia ixx="0.82582" ixy="-0.0019603" ixz="-0.00043035" iyy="0.92115" iyz="0.0013243" izz="0.2601" />
+      <origin  xyz="0 0 0.13" rpy="0 0 0" />
+      <mass value="25.0" />
+      <inertia ixx=".734" ixy="0" ixz="0" iyy=".734" iyz=".0" izz=".156" />
     </inertial>
     <visual>
@@ -36,32 +36,29 @@
     <parent link="base_link"/>
     <child link="laser_mount_link"/>
-    <origin rpy="0 3.1416 3.1416" xyz=".118 0 .253"/>
+    <origin rpy="0 3.1416 3.1416" xyz=".148 0 .253"/>
   </joint>
   <link name="left_wheel">
     <collision name="collision">
-      <origin xyz="0 0 0" rpy="0 1.5707 1.5707"/>
+      <origin xyz="0 0 0" rpy="0 0 -1.5708"/>
       <geometry>
-        <cylinder radius="0.1" length="0.02"/>
+        <mesh filename="package://xbot2_description/meshes/wheel.dae" />
       </geometry>
     </collision>
     <visual name="left_wheel_visual">
-      <origin xyz="0 0 0" rpy="0 1.5707 1.5707"/>
+      <origin xyz="0 0 0" rpy="0 0 -1.5708"/>
       <geometry>
-        <cylinder radius="0.1" length="0.02"/>
+        <mesh filename="package://xbot2_description/meshes/wheel.dae" />
       </geometry>
     </visual>
     <inertial>
-      <origin xyz="0 0 0" rpy="0 1.5707 1.5707"/>
-      <mass value="5"/>
-      <cylinder_inertia m="5" r="0.1" h="0.05"/>
-      <inertia
-        ixx="1.0" ixy="0.0" ixz="0.0"
-        iyy="1.0" iyz="0.0"
-        izz="1.0"/>
+      <origin xyz="0 0 0" rpy="0 0 -1.5708"/>
+      <mass value="1.5"/>
+      <cylinder_inertia m="1.5" r="0.09" h="0.05"/>
+      <inertia ixx=".00335" ixy="0" ixz="0" iyy=".006" iyz="0" izz=".00335" />
     </inertial>
   </link>
   <joint type="continuous" name="left_wheel_hinge">
     <axis xyz="0 1 0" rpy="0 0 0"/>
-    <origin xyz="0 0.3 0.08" rpy="0 0 0"/>
+    <origin xyz="0 0.25 .0953" rpy="0 0 0"/>
     <parent link="base_link"/>
     <child link="left_wheel"/>
@@ -70,28 +67,25 @@
   <link name="right_wheel">
     <collision name="collision">
-      <origin xyz="0 0 0" rpy="0 1.5707 1.5707"/>
+      <origin xyz="0 0 0" rpy="0 0 1.5708 "/>
       <geometry>
-        <cylinder radius="0.1" length="0.02"/>
+        <mesh filename="package://xbot2_description/meshes/wheel.dae" />
       </geometry>
     </collision>
     <visual name="right_wheel_visual">
-      <origin xyz="0 0 0" rpy="0 1.5707 1.5707"/>
+      <origin xyz="0 0 0" rpy="0 0 1.5708"/>
       <geometry>
-        <cylinder radius="0.1" length="0.02"/>
+        <mesh filename="package://xbot2_description/meshes/wheel.dae" />
       </geometry>
     </visual>
     <inertial>
-      <origin xyz="0 0 0" rpy="0 1.5707 1.5707"/>
-      <mass value="5"/>
-      <cylinder_inertia m="5" r="0.1" h="0.05"/>
-      <inertia
-        ixx="1.0" ixy="0.0" ixz="0.0"
-        iyy="1.0" iyz="0.0"
-        izz="1.0"/>
+      <origin xyz="0 0 0" rpy="0 0 1.5708"/>
+      <mass value="1.5"/>
+      <cylinder_inertia m="1.5" r="0.09" h="0.05"/>
+      <inertia ixx=".00335" ixy="0" ixz="0" iyy=".006" iyz="0" izz=".00335" />
     </inertial>
   </link>
   <joint type="continuous" name="right_wheel_hinge">
     <axis xyz="0 1 0" rpy="0 0 0"/>
-    <origin xyz="0 -0.3 0.08" rpy="0 0 0"/>
+    <origin xyz="0 -0.25 .0953" rpy="0 0 0"/>
     <parent link="base_link"/>
     <child link="right_wheel"/>
@@ -100,7 +94,7 @@
   <link name="yaw_platform">
     <inertial>
-      <origin  xyz="-0.0033678 -0.047443 0.62953" rpy="0 0 0" />
-      <mass value=".109" />
-      <inertia ixx="0.82582" ixy="-0.0019603" ixz="-0.00043035" iyy="0.92115" iyz="0.0013243" izz="0.2601" />
+      <origin  xyz="0 0 0" rpy="0 0 0" />
+      <mass value=".11" />
+      <inertia ixx="0.000826" ixy="0" ixz="0" iyy="0.0009211" iyz="0" izz="0.0002601" />
     </inertial>
     <visual>
@@ -124,9 +118,9 @@
     <limit effort="100" velocity="100" lower="-1.57" upper="1.57" />
   </joint>
-  <link name="pitch_platform">
+  <!--link name="pitch_platform">
     <inertial>
       <origin  xyz="-0.0033678 -0.047443 0.62953" rpy="0 0 0" />
-      <mass value=".109" />
-      <inertia ixx="0.82582" ixy="-0.0019603" ixz="-0.00043035" iyy="0.92115" iyz="0.0013243" izz="0.2601" />
+      <mass value=".05" />
+      <inertia ixx="0.0001" ixy="0" ixz="0" iyy="0.00001" iyz="0" izz="0.0001" />
     </inertial>
     <visual>
@@ -142,6 +136,6 @@
       </geometry>
     </collision>
-  </link>
-  <joint name="yaw_to_pitch_platform" type="revolute">
+  </link -->
+  <!-- joint name="yaw_to_pitch_platform" type="revolute">
     <axis xyz="0 1 0"/>
     <parent link="yaw_platform"/>
@@ -149,5 +143,5 @@
     <origin rpy="0 0 0" xyz="0 0 .08"/>
     <limit effort="100" velocity="100" lower="-1.57" upper="1.57" />
-  </joint>
+  </joint -->
   </xacro:macro>
 </robot>

Commit message: type: fix better support for cmd control and yaw control

File: urdf/sick_tim.urdf.xacro (robot description, xacro)
@@ -58,5 +58,5 @@
     <gazebo reference="${link}">
       <material value="Gazebo/LightWood" />
-      <sensor type="ray" name="${name}">
+      <sensor type="gpu_ray" name="${name}">
         <always_on>true</always_on>
         <update_rate>${update_rate}</update_rate>
@@ -78,5 +78,5 @@
           </range>
         </ray>
-        <plugin name="gazebo_ros_${name}_controller" filename="libgazebo_ros_laser.so">
+        <plugin name="gazebo_ros_${name}_controller" filename="libgazebo_ros_gpu_laser.so">
           <gaussianNoise>0.01</gaussianNoise>
           <alwaysOn>true</alwaysOn>

File: urdf/xbot2.urdf.xacro (robot description, xacro)
@@ -60,5 +60,5 @@
   <joint type="continuous" name="left_wheel_hinge">
     <axis xyz="0 1 0" rpy="0 0 0"/>
-    <origin xyz="0 0.25 .0953" rpy="0 0 0"/>
+    <origin xyz="0 0.25 .095" rpy="0 0 0"/>
     <parent link="base_link"/>
     <child link="left_wheel"/>
@@ -87,5 +87,5 @@
   <joint type="continuous" name="right_wheel_hinge">
     <axis xyz="0 1 0" rpy="0 0 0"/>
-    <origin xyz="0 -0.25 .0953" rpy="0 0 0"/>
+    <origin xyz="0 -0.25 .095" rpy="0 0 0"/>
     <parent link="base_link"/>
     <child link="right_wheel"/>

Commit message: move meshes/ into model/meshes/

File: urdf/sick_tim.urdf.xacro (robot description, xacro)
@@ -8,5 +8,5 @@
       length="0.06" width="0.06" height="0.079" mass="0.150" z_offset="0.05595"
       min_range="0.05" max_range="4.0"
-      mesh="package://xbot2_description/meshes/sick_tim310.stl" />
+      mesh="package://xbot2_description/models/meshes/sick_tim310.stl" />
   </xacro:macro>
   <xacro:macro name="sick_tim551" params="name ros_topic">
@@ -14,5 +14,5 @@
       length="0.06" width="0.06" height="0.086" mass="0.250" z_offset="0.06296"
       min_range="0.05" max_range="10.0"
-      mesh="package://xbot2_description/meshes/sick_tim551.stl" />
+      mesh="package://xbot2_description/models/meshes/sick_tim551.stl" />
   </xacro:macro>
   <xacro:macro name="sick_tim571" params="name ros_topic">
@@ -20,5 +20,5 @@
       length="0.06" width="0.06" height="0.086" mass="0.250" z_offset="0.02"
       min_range="0.05" max_range="25.0"
-      mesh="package://xbot2_description/meshes/sick_tim571.stl" />
+      mesh="package://xbot2_description/models/meshes/sick_tim571.stl" />
   </xacro:macro>
   <xacro:macro name="sick_tim" params="name ros_topic length width height mass z_offset min_range max_range mesh">

File: urdf/xbot2.urdf.xacro (robot description, xacro)
@@ -21,5 +21,5 @@
       <origin xyz="0 0 0" rpy="0 0 0" />
       <geometry>
-        <mesh filename="package://xbot2_description/meshes/base_link.dae" />
+        <mesh filename="package://xbot2_description/models/meshes/base_link.dae" />
       </geometry>
     </visual>
@@ -78,5 +78,5 @@
       <origin xyz="0 0 0" rpy="0 0 -1.570796"/>
       <geometry>
-        <mesh filename="package://xbot2_description/meshes/wheel.dae" />
+        <mesh filename="package://xbot2_description/models/meshes/wheel.dae" />
       </geometry>
     </visual>
@@ -105,5 +105,5 @@
       <origin xyz="0 0 0" rpy="0 0 1.570796"/>
       <geometry>
-        <mesh filename="package://xbot2_description/meshes/wheel.dae" />
+        <mesh filename="package://xbot2_description/models/meshes/wheel.dae" />
       </geometry>
     </visual>
@@ -131,5 +131,5 @@
       <origin xyz="0 0 0" rpy="0 0 1.570796" />
       <geometry>
-        <mesh filename="package://xbot2_description/meshes/yaw_platform.stl" />
+        <mesh filename="package://xbot2_description/models/meshes/yaw_platform.stl" />
       </geometry>
       <material name="grey"/>
@@ -159,5 +159,5 @@
       <origin xyz="0 0 0" rpy="0 0 0" />
       <geometry>
-        <mesh filename="package://xbot2_description/meshes/pitch_platform.stl" />
+        <mesh filename="package://xbot2_description/models/meshes/pitch_platform.stl" />
       </geometry>
       <material name="grey"/>
@@ -189,5 +189,5 @@
       <origin xyz="0 0 0" rpy="0 0 0"/>
       <geometry>
-        <mesh filename="package://xbot2_description/meshes/xtion_pro_camera.dae" />
+        <mesh filename="package://xbot2_description/models/meshes/xtion_pro_camera.dae" />
       </geometry>
       <material name="gray"/>
