Commit message: type: feat add the pitch platform

File: urdf/xbot2.urdf.xacro (robot description, xacro)
@@ -118,30 +118,30 @@
     <limit effort="100" velocity="100" lower="-1.57" upper="1.57" />
   </joint>
-  <!--link name="pitch_platform">
+  <link name="pitch_platform">
     <inertial>
-      <origin  xyz="-0.0033678 -0.047443 0.62953" rpy="0 0 0" />
+      <origin  xyz="0 0 0" rpy="0 0 0" />
       <mass value=".05" />
       <inertia ixx="0.0001" ixy="0" ixz="0" iyy="0.00001" iyz="0" izz="0.0001" />
     </inertial>
     <visual>
-      <origin xyz="0 0 0" rpy="0 3.1416 1.5708" />
+      <origin xyz="0 0 0" rpy="0 0 0" />
       <geometry>
-        <mesh filename="package://xbot2_description/meshes/pitch_platform.dae" />
+        <mesh filename="package://xbot2_description/meshes/pitch_platform.stl" />
       </geometry>
     </visual>
     <collision>
-      <origin xyz="0 0 0" rpy="0 3.1416 1.5708" />
+      <origin xyz="0 0 0" rpy="0 0 0" />
       <geometry>
-        <mesh filename="package://xbot2_description/meshes/pitch_platform.dae" />
+        <mesh filename="package://xbot2_description/meshes/pitch_platform.stl" />
       </geometry>
     </collision>
-  </link -->
-  <!-- joint name="yaw_to_pitch_platform" type="revolute">
+  </link>
+  <joint name="yaw_to_pitch_platform" type="revolute">
     <axis xyz="0 1 0"/>
     <parent link="yaw_platform"/>
     <child link="pitch_platform"/>
-    <origin rpy="0 0 0" xyz="0 0 .08"/>
+    <origin rpy="0 0 0" xyz="0 0 .02"/>
     <limit effort="100" velocity="100" lower="-1.57" upper="1.57" />
-  </joint -->
+  </joint>
   </xacro:macro>
 </robot>

Commit message: type: feat add RGBD camera on top of xbot2

File: urdf/xbot2.urdf.xacro (robot description, xacro)
@@ -144,4 +144,42 @@
     <limit effort="100" velocity="100" lower="-1.57" upper="1.57" />
   </joint>
+  <!-- Camera -->
+  <link name="camera_link">
+    <collision>
+      <origin xyz="0 0 0" rpy="0 0 0"/>
+      <geometry>
+        <mesh filename="package://xbot2_description/meshes/xtion_pro_camera.dae" />
+      </geometry>
+    </collision>
+    <visual>
+      <origin xyz="0 0 0" rpy="0 0 0"/>
+      <geometry>
+        <mesh filename="package://xbot2_description/meshes/xtion_pro_camera.dae" />
+      </geometry>
+      <material name="red"/>
+    </visual>
+    <inertial>
+      <mass value="1e-5" />
+      <origin xyz="0 0 0" rpy="0 0 0"/>
+      <inertia ixx="1e-6" ixy="0" ixz="0" iyy="1e-6" iyz="0" izz="1e-6" />
+    </inertial>
+  </link>
+  <joint name="camera_joint" type="fixed">
+    <axis xyz="0 1 0" />
+    <origin xyz="0 0 0" rpy="0 0 0"/>
+    <parent link="pitch_platform"/>
+    <child link="camera_link"/>
+  </joint>
+  <!-- generate an optical frame http://www.ros.org/reps/rep-0103.html#suffix-frames
+      so that ros and opencv can operate on the camera frame correctly -->
+  <joint name="camera_optical_joint" type="fixed">
+    <!-- these values have to be these values otherwise the gazebo camera image
+        won't be aligned properly with the frame it is supposedly originating from -->
+    <origin xyz="0 0 0" rpy="${-pi/2} 0 ${-pi/2}"/>
+    <parent link="camera_link"/>
+    <child link="camera_link_optical"/>
+  </joint>
+  <link name="camera_link_optical">
+  </link>
   </xacro:macro>
 </robot>

Commit message: type: fix fix some bugs

File: urdf/xbot2.urdf.xacro (robot description, xacro)
@@ -40,7 +40,7 @@
   <link name="left_wheel">
     <collision name="collision">
-      <origin xyz="0 0 0" rpy="0 0 -1.5708"/>
+      <origin xyz="0 0 0" rpy="1.5708 0 0"/>
       <geometry>
-        <mesh filename="package://xbot2_description/meshes/wheel.dae" />
+        <cylinder radius="0.095" length="0.04"/>
       </geometry>
     </collision>
@@ -54,20 +54,20 @@
       <origin xyz="0 0 0" rpy="0 0 -1.5708"/>
       <mass value="1.5"/>
-      <cylinder_inertia m="1.5" r="0.09" h="0.05"/>
-      <inertia ixx=".00335" ixy="0" ixz="0" iyy=".006" iyz="0" izz=".00335" />
+      <inertia ixx=".001" ixy="0" ixz="0" iyy=".001" iyz="0" izz=".001" />
     </inertial>
   </link>
   <joint type="continuous" name="left_wheel_hinge">
     <axis xyz="0 1 0" rpy="0 0 0"/>
-    <origin xyz="0 0.25 .095" rpy="0 0 0"/>
+    <origin xyz="0 0.245 .095" rpy="0 0 0"/>
     <parent link="base_link"/>
     <child link="left_wheel"/>
+    <limit effort="100000" velocity="1000"/>
     <joint_properties damping="0.0" friction="0.0"/>
   </joint>
   <link name="right_wheel">
     <collision name="collision">
-      <origin xyz="0 0 0" rpy="0 0 1.5708 "/>
+      <origin xyz="0 0 0" rpy="-1.5708  0 0"/>
       <geometry>
-        <mesh filename="package://xbot2_description/meshes/wheel.dae" />
+        <cylinder radius="0.095" length="0.04"/>
       </geometry>
     </collision>
@@ -81,13 +81,13 @@
       <origin xyz="0 0 0" rpy="0 0 1.5708"/>
       <mass value="1.5"/>
-      <cylinder_inertia m="1.5" r="0.09" h="0.05"/>
-      <inertia ixx=".00335" ixy="0" ixz="0" iyy=".006" iyz="0" izz=".00335" />
+      <inertia ixx=".001" ixy="0" ixz="0" iyy=".001" iyz="0" izz=".001" />
     </inertial>
   </link>
   <joint type="continuous" name="right_wheel_hinge">
     <axis xyz="0 1 0" rpy="0 0 0"/>
-    <origin xyz="0 -0.25 .095" rpy="0 0 0"/>
+    <origin xyz="0 -0.245 .095" rpy="0 0 0"/>
     <parent link="base_link"/>
     <child link="right_wheel"/>
+    <limit effort="100000" velocity="1000"/>
     <joint_properties damping="0.0" friction="0.0"/>
   </joint>

Commit message: replace collision model with simple shapes to lessen computation

File: urdf/xbot2.urdf.xacro (robot description, xacro)
@@ -14,7 +14,7 @@
   <link name="base_link">
     <inertial>
-      <origin  xyz="0 0 0.13" rpy="0 0 0" />
-      <mass value="25.0" />
-      <inertia ixx=".734" ixy="0" ixz="0" iyy=".734" iyz=".0" izz=".156" />
+      <origin  xyz="0.001 0 0.007" rpy="0 0 0" />
+      <mass value="30.0" />
+      <inertia ixx="1.734" ixy="0" ixz="0" iyy="1.734" iyz=".0" izz="1.0" />
     </inertial>
     <visual>
@@ -24,8 +24,38 @@
       </geometry>
     </visual>
-    <collision>
-      <origin xyz="0 0 0" rpy="0 0 0" />
-      <geometry>
-        <mesh filename="package://xbot2_description/meshes/base_link.dae" />
+    <collision name="front_omniwheel">
+      <origin xyz="0.18 0 0.02" rpy="0 0 0" />
+      <geometry>
+        <sphere radius="0.019"/>
+      </geometry>
+    </collision>
+    <collision name="back_omniwheel">
+      <origin xyz="-0.18 0 0.02" rpy="0 0 0" />
+      <geometry>
+        <sphere radius="0.019"/>
+      </geometry>
+    </collision>
+    <collision name="collision1">
+      <origin xyz="0.0 0 0.135" rpy="0 0 0" />
+      <geometry>
+        <cylinder length="0.15" radius="0.25"/>
+      </geometry>
+    </collision>
+    <collision name="collision2">
+      <origin xyz="0.03 0 0.25" rpy="0 0 0" />
+      <geometry>
+        <cylinder length="0.08" radius="0.15"/>
+      </geometry>
+    </collision>
+    <collision name="collision3">
+      <origin xyz="0 0 0.68" rpy="0 0 0" />
+      <geometry>
+        <cylinder length="0.8" radius="0.08"/>
+      </geometry>
+    </collision>
+    <collision name="collision4">
+      <origin xyz="0 0 1.135" rpy="0 0 0" />
+      <geometry>
+        <box size="0.04 0.17 0.09"/>
       </geometry>
     </collision>
@@ -40,11 +70,11 @@
   <link name="left_wheel">
     <collision name="collision">
-      <origin xyz="0 0 0" rpy="1.5708 0 0"/>
-      <geometry>
-        <cylinder radius="0.095" length="0.04"/>
+      <origin xyz="0 0 0" rpy="1.570796 0 0"/>
+      <geometry>
+        <cylinder radius="0.095" length="0.05"/>
       </geometry>
     </collision>
     <visual name="left_wheel_visual">
-      <origin xyz="0 0 0" rpy="0 0 -1.5708"/>
+      <origin xyz="0 0 0" rpy="0 0 -1.570796"/>
       <geometry>
         <mesh filename="package://xbot2_description/meshes/wheel.dae" />
@@ -52,5 +82,5 @@
     </visual>
     <inertial>
-      <origin xyz="0 0 0" rpy="0 0 -1.5708"/>
+      <origin xyz="0 0 0" rpy="0 0 -1.570796"/>
       <mass value="1.5"/>
       <inertia ixx=".001" ixy="0" ixz="0" iyy=".001" iyz="0" izz=".001" />
@@ -67,11 +97,11 @@
   <link name="right_wheel">
     <collision name="collision">
-      <origin xyz="0 0 0" rpy="-1.5708  0 0"/>
-      <geometry>
-        <cylinder radius="0.095" length="0.04"/>
+      <origin xyz="0 0 0" rpy="-1.570796  0 0"/>
+      <geometry>
+        <cylinder radius="0.095" length="0.05"/>
       </geometry>
     </collision>
     <visual name="right_wheel_visual">
-      <origin xyz="0 0 0" rpy="0 0 1.5708"/>
+      <origin xyz="0 0 0" rpy="0 0 1.570796"/>
       <geometry>
         <mesh filename="package://xbot2_description/meshes/wheel.dae" />
@@ -79,5 +109,5 @@
     </visual>
     <inertial>
-      <origin xyz="0 0 0" rpy="0 0 1.5708"/>
+      <origin xyz="0 0 0" rpy="0 0 1.570796"/>
       <mass value="1.5"/>
       <inertia ixx=".001" ixy="0" ixz="0" iyy=".001" iyz="0" izz=".001" />
@@ -99,5 +129,5 @@
     </inertial>
     <visual>
-      <origin xyz="0 0 0" rpy="0 0 1.5708" />
+      <origin xyz="0 0 0" rpy="0 0 1.570796" />
       <geometry>
         <mesh filename="package://xbot2_description/meshes/yaw_platform.stl" />
@@ -106,7 +136,7 @@
     </visual>
     <collision>
-      <origin xyz="0 0 0" rpy="0 0 1.5708" />
-      <geometry>
-        <mesh filename="package://xbot2_description/meshes/yaw_platform.stl" />
+      <origin xyz="0 0 0" rpy="0 0 1.570796" />
+      <geometry>
+        <box size="0.0 0.0 0.0"/>
       </geometry>
     </collision>
@@ -136,5 +166,5 @@
       <origin xyz="0 0 0" rpy="0 0 0" />
       <geometry>
-        <mesh filename="package://xbot2_description/meshes/pitch_platform.stl" />
+        <box size="0.0 0.0 0.0"/>
       </geometry>
     </collision>
@@ -153,5 +183,5 @@
       <origin xyz="0 0 0" rpy="0 0 0"/>
       <geometry>
-        <mesh filename="package://xbot2_description/meshes/xtion_pro_camera.dae" />
+        <box size="0.0 0.0 0.0"/>
       </geometry>
     </collision>

Commit message: fix: replace some collision geometry of (0,0,0) with (0.01,0.01,0.01)

File: urdf/xbot2.urdf.xacro (robot description, xacro)
@@ -138,5 +138,5 @@
       <origin xyz="0 0 0" rpy="0 0 1.570796" />
       <geometry>
-        <box size="0.0 0.0 0.0"/>
+        <box size="0.01 0.01 0.01"/>
       </geometry>
     </collision>
@@ -166,5 +166,5 @@
       <origin xyz="0 0 0" rpy="0 0 0" />
       <geometry>
-        <box size="0.0 0.0 0.0"/>
+        <box size="0.01 0.01 0.01"/>
       </geometry>
     </collision>
@@ -183,5 +183,5 @@
       <origin xyz="0 0 0" rpy="0 0 0"/>
       <geometry>
-        <box size="0.0 0.0 0.0"/>
+        <box size="0.01 0.01 0.01"/>
       </geometry>
     </collision>

Commit message: revert laserscan 180 degrees

File: urdf/xbot2.urdf.xacro (robot description, xacro)
@@ -66,5 +66,5 @@
     <parent link="base_link"/>
     <child link="laser_mount_link"/>
-    <origin rpy="0 3.1416 3.1416" xyz=".148 0 .253"/>
+    <origin rpy="3.1416 3.1416 3.1416" xyz=".148 0 .253"/>
   </joint>
   <link name="left_wheel">

Commit message: modify collision model

File: urdf/xbot2.urdf.xacro (robot description, xacro)
@@ -45,5 +45,5 @@
       <origin xyz="0.03 0 0.25" rpy="0 0 0" />
       <geometry>
-        <cylinder length="0.08" radius="0.15"/>
+        <cylinder length="0.08" radius="0.04"/>
       </geometry>
     </collision>
